Commit message: fixed directories for the urdf

File: URDF/new_mycobot_pro_320.urdf (robot description, URDF)
Before this commit: robot firefighter, 7 links, 6 joints
Links:
- link base: geometry collision mesh filename=base.dae; visual mesh filename=base.dae
- link link1: geometry collision mesh filename=link1.dae; visual mesh filename=link1.dae
- link link2: geometry collision mesh filename=link2.dae; visual mesh filename=link2.dae
- link link3: geometry collision mesh filename=link3.dae; visual mesh filename=link3.dae
- link link4: geometry collision mesh filename=link4.dae; visual mesh filename=link4.dae
- link link5: geometry collision mesh filename=link5.dae; visual mesh filename=link5.dae
- link link6: geometry collision mesh filename=link6.dae; visual mesh filename=link6.dae

Commit message: basic operation is available

File: URDF/new_mycobot_pro_320.urdf (robot description, URDF)
Before this commit: robot firefighter, 7 links, 6 joints
Links:
- link base: geometry collision mesh filename=base.dae; visual mesh filename=base.dae scale=0.001 0.001 0.001
- link link1: geometry collision mesh filename=link1.dae scale=0.001 0.001 0.001; visual mesh filename=link1.dae scale=0.001 0.001 0.001
- link link2: geometry collision mesh filename=link2.dae scale=0.001 0.001 0.001; visual mesh filename=link2.dae scale=0.001 0.001 0.001
- link link3: geometry collision mesh filename=link3.dae scale=0.001 0.001 0.001; visual mesh filename=link3.dae scale=0.001 0.001 0.001
- link link4: geometry collision mesh filename=link4.dae scale=0.001 0.001 0.001; visual mesh filename=link4.dae scale=0.001 0.001 0.001
- link link5: geometry collision mesh filename=link5.dae scale=0.001 0.001 0.001; visual mesh filename=link5.dae scale=0.001 0.001 0.001
- link link6: geometry collision mesh filename=link6.dae scale=0.001 0.001 0.001; visual mesh filename=link6.dae scale=0.001 0.001 0.001
